File: gg.kicad_pcb (KiCad board)
At the start: 2 copper layers, 70 parts, among them J1 USB_B_Micro, J10 Screw, J11 Screw, J12 A, J13 Micro, J14 Speaker, J15 A, J16 A, J17 i2c, J18 i2c, J2 AVR-ISP-6, J3 Screw, J4 pwm, J5 pwm, J6 pwm, J7 Screw, J8 Screw, J9 Screw, K1 SRD, K2 SRD, K3 SRD, K4 SRD, K5 SRD, K6 SRD, Q1 2N3904, Q2 2N3904, Q3 2N3904, Q4 2N3904, Q5 2N3904, Q6 2N3904, U1 PC817, U2 PC817, U3 PC817, U4 ATmega328P-PU, U5 Sim800l, U6 PC817, U7 PC817, U8 PC817, Y1 Crystal

Commit message: 1.2.0
Parts:
- moved J7 163.1 mm to (24.5, 77.3), turned to 270 degrees
- moved Q4 154.6 mm to (53.0, 111.3), turned to 270 degrees
- moved U6 153.6 mm to (63.7, 119.1), turned to 180 degrees
- moved Q6 147.9 mm to (53.0, 24.1), turned to 270 degrees
- moved J3 144.7 mm to (24.5, 59.9), turned to 270 degrees
- moved Q5 143.7 mm to (53.0, 41.5), turned to 270 degrees
- moved J8 142.4 mm to (24.5, 95.0), turned to 270 degrees
- moved Q2 142.2 mm to (53.0, 75.9), turned to 270 degrees
- moved D5 139.3 mm to (52.8, 117.5), turned to 270 degrees
- moved R15 138.6 mm to (56.9, 24.1)
- moved R11 133.1 mm to (56.9, 110.9)
- moved C8 132.7 mm to (72.0, 89.2), turned to 270 degrees
- moved D7 131.2 mm to (52.8, 30.5), turned to 270 degrees
- moved R12 130.9 mm to (56.9, 54.5)
- moved J11 130.8 mm to (24.5, 25.4), turned to 270 degrees
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Connections:
- J6 pad 2: P17 -> MOSI
Routing:
- net +5V: track 0.00 -> 105.8 mm
- net Net-(J8-Pad2): track 0.00 -> 23.8 mm
- net Net-(J3-Pad2): track 0.00 -> 23.8 mm
- net Net-(J9-Pad2): track 0.00 -> 23.8 mm
- net Net-(J7-Pad2): track 0.00 -> 23.8 mm
- net Net-(J10-Pad2): track 0.00 -> 23.7 mm
- net Net-(J11-Pad2): track 0.00 -> 23.7 mm
- net GND: track 0.00 -> 21.1 mm
- net Net-(C8-Pad2): track 0.00 -> 11.9 mm
- net Net-(D3-Pad1): track 0.00 -> 11.6 mm
- net Net-(D7-Pad1): track 0.00 -> 11.5 mm
- net Net-(D1-Pad1): track 0.00 -> 11.4 mm
- net Net-(D4-Pad1): track 0.00 -> 11.3 mm
- net Net-(D5-Pad1): track 0.00 -> 11.2 mm
- net Net-(D6-Pad1): track 0.00 -> 11.1 mm
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
Commit message: 1.3.0
Parts:
- removed C5: 100nf, Capacitor_THT:C_Disc_D5.0mm_W2.5mm_P2.50mm
- moved J13 97.0 mm to (126.9, 122.2), turned to 180 degrees
- moved J14 94.9 mm to (116.0, 122.2), turned to 180 degrees
- moved C4 45.0 mm to (78.4, 79.5), turned to 180 degrees
- moved C3 38.3 mm to (93.6, 82.2)
- moved U5 25.9 mm to (110.2, 33.1)
- moved D8 23.4 mm to (66.9, 23.7), turned to 270 degrees
- moved C1 22.3 mm to (88.3, 33.7)
- moved C6 22.0 mm to (93.6, 85.3)
- moved R5 21.7 mm to (82.0, 38.2), turned to 270 degrees
- moved J6 18.6 mm to (95.4, 95.0), turned to 90 degrees
- moved J12 17.4 mm to (95.4, 67.2), turned to 90 degrees
- moved D2 15.8 mm to (88.8, 29.5), turned to 180 degrees
- moved J5 15.0 mm to (95.4, 104.4), turned to 90 degrees
- moved R4 14.2 mm to (81.9, 46.7), turned to 180 degrees
- moved J16 12.6 mm to (95.4, 75.9), turned to 90 degrees
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Connections:
- J12 pad 1: +5V -> A2
- J12 pad 2: A2 -> +5V
- J15 pad 1: +5V -> A1
- J15 pad 2: A1 -> +5V
- J16 pad 1: +5V -> A0
- J16 pad 2: A0 -> +5V
- J2 pad 2: +5V -> MOSI
- J2 pad 4: MOSI -> +5V
- J4 pad 1: +5V -> P16
- J4 pad 2: P16 -> +5V
- J5 pad 1: +5V -> P15
- J5 pad 2: P15 -> +5V
- J6 pad 1: +5V -> MOSI
- J6 pad 2: MOSI -> +5V
- U1 pad 2: D11 -> D6
- U7 pad 2: D6 -> D5
- U8 pad 2: D5 -> D4
Routing:
- net RST: track 0.00 -> 110.8 mm
- net GND: track 21.1 -> 89.9 mm
- net +5V: track 105.8 -> 162.6 mm
- net D4: track 0.00 -> 55.1 mm
- net D5: track 0.00 -> 43.2 mm
- net TXD: track 0.00 -> 39.7 mm
- net D12: track 0.00 -> 30.4 mm
- net D6: track 0.00 -> 29.1 mm
- net D14: track 0.00 -> 26.4 mm
- net RXD: track 0.00 -> 25.5 mm
- net RXD3v3: track 0.00 -> 24.5 mm
- net SCL: track 0.00 -> 21.8 mm
- net SDA: track 0.00 -> 20.8 mm
- net D13: track 0.00 -> 20.1 mm
- net MOSI: track 0.00 -> 16.6 mm
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
Commit message: 1.4.0
Parts:
- moved D8 15.0 mm to (73.5, 37.2), turned to 90 degrees
- moved R16 3.63 mm to (78.6, 32.3)
- moved R6 3.33 mm to (55.9, 87.1)
- moved R8 3.20 mm to (55.9, 122.3)
- moved R1 3.08 mm to (55.9, 69.7)
- moved J4 3.05 mm to (96.3, 102.6)
- moved J6 3.05 mm to (96.3, 97.9)
- moved J5 3.05 mm to (96.3, 107.3)
- moved R7 2.96 mm to (55.9, 105.0)
- moved C4 2.82 mm to (76.7, 77.2), turned to 270 degrees
- moved R14 2.80 mm to (56.0, 35.4)
- moved R10 2.34 mm to (57.4, 91.1), turned to 270 degrees
- moved R11 2.21 mm to (57.4, 108.7), turned to 270 degrees
- moved R13 2.19 mm to (57.4, 39.2), turned to 270 degrees
- moved R2 2.09 mm to (57.4, 56.1), turned to 270 degrees
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Connections:
- J2 pad 5: RST -> GND
- J2 pad 6: GND -> RST
Routing:
- net +5V: track 162.6 -> 407.4 mm
- net RST: track 110.8 -> 48.8 mm
- net GND: track 89.9 -> 100.2 mm
- net D5: track 43.2 -> 37.6 mm
- net Net-(R13-Pad2): track 8.18 -> 3.10 mm
- net Net-(R9-Pad2): track 8.26 -> 3.20 mm
- net Net-(R2-Pad2): track 8.26 -> 3.20 mm
- net Net-(R11-Pad2): track 8.26 -> 3.33 mm
- net D6: track 29.1 -> 24.2 mm
- net Net-(R10-Pad2): track 8.26 -> 3.46 mm
- net P15: track 10.9 -> 14.6 mm
- net Net-(D8-Pad2): track 5.34 -> 2.41 mm
- net Net-(R6-Pad2): track 7.21 -> 4.45 mm
- net MOSI: track 16.6 -> 19.4 mm
- net D4: track 55.1 -> 52.4 mm
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
Commit message: 2.0.0
Parts:
- added H1: MountingHole, MountingHole:MountingHole_2.7mm_M2.5_Pad_Via, F.Cu at (120.0, 17.0)
- added H2: MountingHole, MountingHole:MountingHole_2.7mm_M2.5_Pad_Via, F.Cu at (25.0, 17.0)
- added H3: MountingHole, MountingHole:MountingHole_2.7mm_M2.5_Pad_Via, F.Cu at (120.0, 130.0)
- added H4: MountingHole, MountingHole:MountingHole_2.7mm_M2.5_Pad_Via, F.Cu at (25.0, 130.0)
- added J19: Micro, TerminalBlock:TerminalBlock_bornier-2_P5.08mm, F.Cu at (91.6, 22.1)
- added J20: Micro, TerminalBlock:TerminalBlock_bornier-2_P5.08mm, F.Cu at (118.9, 75.8)
- J2: value AVR-ISP-6 -> Screw_Terminal_01x04; footprint Connector_PinSocket_2.54mm:PinSocket_2x03_P2.54mm_Vertical -> TerminalBlock:TerminalBlock_bornier-4_P5.08mm
- moved J14 68.8 mm to (118.9, 53.5), turned to 90 degrees
- moved J13 58.3 mm to (118.9, 64.4), turned to 90 degrees
- moved J4 22.1 mm to (116.3, 111.9)
- moved J5 22.1 mm to (116.3, 116.6)
- moved J6 22.1 mm to (116.3, 107.2)
- moved J2 20.8 mm to (118.8, 82.6), turned to 270 degrees
Connections:
- J2 pad 1: MISO -> 14
- J2 pad 2: MOSI -> SCK
- J2 pad 3: SCK -> MISO
- J2 pad 4: +5V -> Net-(J2-Pad4)
- U4 pad 23: A0 -> 14
- U4 pad 24: A1 -> A0
- U4 pad 25: A2 -> A1
- U4 pad 26: Net-(U4-Pad26) -> A2
Routing:
- net +5V: track 407.4 -> 481.9 mm
- net Net-(J13-Pad1): track 0.00 -> 47.7 mm
- net Net-(J13-Pad2): track 0.00 -> 35.7 mm
- net 14: track 0.00 -> 31.0 mm
- net P16: track 9.87 -> 33.8 mm
- net P15: track 14.6 -> 38.6 mm
- net Net-(J14-Pad1): track 0.00 -> 23.6 mm
- net MISO: track 9.58 -> 29.9 mm
- net SCK: track 9.58 -> 28.9 mm
- net MOSI: track 19.4 -> 34.9 mm
- net Net-(J14-Pad2): track 0.00 -> 7.18 mm
- net GND: track 100.2 -> 98.0 mm
- net A2: track 8.27 -> 6.62 mm
- net A1: track 7.39 -> 5.86 mm
- added copper zone on F.Cu, net GND
Other:
- board outline added: 105 x 123 mm

Commit message: 2.2.0
Parts:
- added J21: Conn_02x04_Odd_Even, Connector_PinSocket_2.54mm:PinSocket_2x04_P2.54mm_Vertical, F.Cu at (106.9, 33.7)
- added J22: Conn_01x02_Male, Connector_PinHeader_2.54mm:PinHeader_1x02_P2.54mm_Vertical, F.Cu at (72.2, 45.5)
Connections:
- net Net-(C1-Pad1) renamed 3v3
Routing:
- net 3v3: track 15.0 -> 73.5 mm
- net RST: track 48.8 -> 96.5 mm
- net RXD3v3: track 24.5 -> 47.4 mm
- net GND: track 98.0 -> 117.8 mm
- net TXD: track 39.7 -> 49.4 mm
Other:
- board text added: "Safta IOT"
