File: gg.sch (KiCad schematic (older format))
At the start: 70 parts, among them J1 USB_B_Micro, J10 Screw, J11 Screw, J12 A, J13 Micro, J14 Speaker, J15 A, J16 A, J17 i2c, J18 i2c, J2 AVR-ISP-6, J3 Screw, J4 pwm, J5 pwm, J6 pwm, J7 Screw, J8 Screw, J9 Screw, K1 SRD, K2 SRD, K3 SRD, K4 SRD, K5 SRD, K6 SRD, Q1 2N3904, Q2 2N3904, Q3 2N3904, Q4 2N3904, Q5 2N3904, Q6 2N3904, U1 PC817, U2 PC817, U3 PC817, U4 ATmega328P-PU, U5 Sim800l, U6 PC817, U7 PC817, U8 PC817, Y1 Crystal

Commit message: 1.2.0
Connections:
- wire segments 214 -> 215
Changed lines of the file:
@@
 Text GLabel 6150 1850 2    50   Input ~ 0
 P16
-Text GLabel 6650 1750 2    50   Input ~ 0
+Text GLabel 6800 1750 2    50   Input ~ 0
 P17
 Text GLabel 6650 1750 0    50   Input ~ 0
@@
 Wire Wire Line
 	10300 5450 10300 5700
+Wire Wire Line
+	6650 1750 6800 1750
 $EndSCHEMATC

Commit message: 1.3.0
Parts:
- removed C5: 100nf, Capacitor_THT:C_Disc_D5.0mm_W2.5mm_P2.50mm, symbol Device:C
Connections:
- wire segments 215 -> 225
Other:
- moved on the sheet: J12, J15, J16, J4, J5, J6

Commit message: 1.4.0
Changed lines of the file:
@@
 Text GLabel 10800 5050 2    50   Input ~ 0
 SCK
-Text GLabel 10800 5150 2    50   Input ~ 0
+Text GLabel 10300 5700 2    50   Input ~ 0
 RST
 $Comp
 L power:GND #PWR0114
 U 1 1 60BFDF12
-P 10300 5700
-F 0 "#PWR0114" H 10300 5450 50  0001 C CNN
-F 1 "GND" H 10305 5527 50  0000 C CNN
-F 2 "" H 10300 5700 50  0001 C CNN
-F 3 "" H 10300 5700 50  0001 C CNN
-	1    10300 5700
+P 10800 5150
+F 0 "#PWR0114" H 10800 4900 50  0001 C CNN
+F 1 "GND" H 10805 4977 50  0000 C CNN
+F 2 "" H 10800 5150 50  0001 C CNN
+F 3 "" H 10800 5150 50  0001 C CNN
+	1    10800 5150
 	1    0    0    -1
 $EndComp

Commit message: 2.0.0
Parts:
- removed J2: AVR-ISP-6, Connector_PinSocket_2.54mm:PinSocket_2x03_P2.54mm_Vertical, symbol Connector:AVR-ISP-6
- added H1, H2, H3, H4: MountingHole, MountingHole:MountingHole_2.7mm_M2.5_Pad_Via, symbol Mechanical:MountingHole
- added J19, J20: Micro, TerminalBlock:TerminalBlock_bornier-2_P5.08mm, symbol Connector:Screw_Terminal_01x02
- added J2: Screw_Terminal_01x04, TerminalBlock:TerminalBlock_bornier-4_P5.08mm, symbol Connector:Screw_Terminal_01x04
Connections:
- net labels added: 14
- wire segments 225 -> 222
- no-connect marks 7 -> 6
Changed lines of the file:
@@
 	1    0    0    -1
 $EndComp
-$Comp
-L Connector:AVR-ISP-6 J2
-U 1 1 60C231E8
-P 10400 5050
-F 0 "J2" H 10071 5146 50  0000 R CNN
-F 1 "AVR-ISP-6" H 10071 5055 50  0000 R CNN
-F 2 "Connector_PinSocket_2.54mm:PinSocket_2x03_P2.54mm_Vertical" V 10150 5100 50  0001 C CNN
-F 3 " ~" H 9125 4500 50  0001 C CNN
-	1    10400 5050
-	1    0    0    -1
-$EndComp
-Text GLabel 10800 4850 2    50   Input ~ 0
-MISO
-Text GLabel 10300 4450 2    50   Input ~ 0
-MOSI
-Text GLabel 10800 5050 2    50   Input ~ 0
-SCK
-Text GLabel 10300 5700 2    50   Input ~ 0
-RST
-$Comp
-L power:GND #PWR0114
-U 1 1 60BFDF12
-P 10800 5150
-F 0 "#PWR0114" H 10800 4900 50  0001 C CNN
-F 1 "GND" H 10805 4977 50  0000 C CNN
-F 2 "" H 10800 5150 50  0001 C CNN
-F 3 "" H 10800 5150 50  0001 C CNN
-	1    10800 5150
-	1    0    0    -1
-$EndComp
-Wire Wire Line
-	10300 4550 10300 4450
 Text GLabel 6150 1950 2    50   Input ~ 0
 MOSI
@@
 F 3 "http://ww1.microchip.com/downloads/en/DeviceDoc/ATmega328_P%20AVR%20MCU%20with%20picoPower%20Technology%20Data%20Sheet%2040001984A.pdf" H 5550 2850 50  0001 C CNN
 	1    5550 2850
-	1    0    0    -1
-$EndComp
-$Comp
-L power:+5V #PWR0115
-U 1 1 60BFEB44
-P 11100 4950
-F 0 "#PWR0115" H 11100 4800 50  0001 C CNN
-F 1 "+5V" H 11115 5123 50  0000 C CNN
-F 2 "" H 11100 4950 50  0001 C CNN
-F 3 "" H 11100 4950 50  0001 C CNN
-	1    11100 4950
 	1    0    0    -1
 $EndComp
@@
 L power:GND #PWR0127
 U 1 1 60C9A063
-P 9750 3800
-F 0 "#PWR0127" H 9750 3550 50  0001 C CNN
-F 1 "GND" H 9755 3627 50  0000 C CNN
-F 2 "" H 9750 3800 50  0001 C CNN
-F 3 "" H 9750 3800 50  0001 C CNN
-	1    9750 3800
+P 9500 5700
+F 0 "#PWR0127" H 9500 5450 50  0001 C CNN
+F 1 "GND" H 9500 5550 50  0000 C CNN
+F 2 "" H 9500 5700 50  0001 C CNN
+F 3 "" H 9500 5700 50  0001 C CNN
+	1    9500 5700
 	1    0    0    -1
 $EndComp
@@
 Text GLabel 8350 3600 2    50   Input ~ 0
 A2
-Text GLabel 6150 2550 2    50   Input ~ 0
+Text GLabel 6150 2650 2    50   Input ~ 0
 A0
-Text GLabel 6150 2650 2    50   Input ~ 0
+Text GLabel 6150 2750 2    50   Input ~ 0
 A1
-Text GLabel 6150 2750 2    50   Input ~ 0
+Text GLabel 6150 2850 2    50   Input ~ 0
 A2
 Text GLabel 6150 3750 2    50   Input ~ 0
@@
 NoConn ~ 9700 1400
 NoConn ~ 9700 1500
-NoConn ~ 6150 2850
-Wire Wire Line
-	10300 5450 10300 5700
 Wire Wire Line
 	6650 1750 6800 1750
@@
 Wire Wire Line
 	5150 700  5900 700
-Wire Wire Line
-	11100 4950 10800 4950
+Text GLabel 9500 5050 0    50   Input ~ 0
+MISO
+Text GLabel 9500 4950 0    50   Input ~ 0
+SCK
+Text GLabel 6150 2550 2    50   Input ~ 0
+14
+Text GLabel 9500 4850 0    50   Input ~ 0
+14
+$Comp
+L Connector:Screw_Terminal_01x04 J2
+U 1 1 60D52FFB
+P 9700 4950
+F 0 "J2" H 9780 4942 50  0000 L CNN
+F 1 "Screw_Terminal_01x04" H 9780 4851 50  0000 L CNN
+F 2 "TerminalBlock:TerminalBlock_bornier-4_P5.08mm" H 9700 4950 50  0001 C CNN
+F 3 "~" H 9700 4950 50  0001 C CNN
+	1    9700 4950
+	1    0    0    -1
+$EndComp
+$Comp
+L Connector:Screw_Terminal_01x02 J19
+U 1 1 60DAB8F0
+P 10550 4150
+F 0 "J19" H 10630 4142 50  0000 L CNN
+F 1 "Micro" H 10630 4051 50  0000 L CNN
+F 2 "TerminalBlock:TerminalBlock_bornier-2_P5.08mm" H 10550 4150 50  0001 C CNN
+F 3 "~" H 10550 4150 50  0001 C CNN
+	1    10550 4150
+	1    0    0    -1
+$EndComp
+$Comp
+L power:+5V #PWR0114
+U 1 1 60DAC02A
+P 10350 4150
+F 0 "#PWR0114" H 10350 4000 50  0001 C CNN
+F 1 "+5V" H 10365 4323 50  0000 C CNN
+F 2 "" H 10350 4150 50  0001 C CNN
+F 3 "" H 10350 4150 50  0001 C CNN
+	1    10350 4150
+	1    0    0    -1
+$EndComp
+$Comp
+L power:GND #PWR0115
+U 1 1 60DAD162
+P 9750 3800
+F 0 "#PWR0115" H 9750 3550 50  0001 C CNN
+F 1 "GND" H 9755 3627 50  0000 C CNN
+F 2 "" H 9750 3800 50  0001 C CNN
+F 3 "" H 9750 3800 50  0001 C CNN
+	1    9750 3800
+	1    0    0    -1
+$EndComp
+$Comp
+L power:GND #PWR0146
+U 1 1 60DAD65B
+P 10350 4250
+F 0 "#PWR0146" H 10350 4000 50  0001 C CNN
+F 1 "GND" H 10355 4077 50  0000 C CNN
+F 2 "" H 10350 4250 50  0001 C CNN
+F 3 "" H 10350 4250 50  0001 C CNN
+	1    10350 4250
+	1    0    0    -1
+$EndComp
+$Comp
+L Connector:Screw_Terminal_01x02 J20
+U 1 1 60CFE3A3
+P 9700 5600
+F 0 "J20" H 9780 5592 50  0000 L CNN
+F 1 "Micro" H 9780 5501 50  0000 L CNN
+F 2 "TerminalBlock:TerminalBlock_bornier-2_P5.08mm" H 9700 5600 50  0001 C CNN
+F 3 "~" H 9700 5600 50  0001 C CNN
+	1    9700 5600
+	1    0    0    -1
+$EndComp
+$Comp
+L power:+5V #PWR0147
+U 1 1 60CFF3A6
+P 9500 5600
+F 0 "#PWR0147" H 9500 5450 50  0001 C CNN
+F 1 "+5V" H 9515 5773 50  0000 C CNN
+F 2 "" H 9500 5600 50  0001 C CNN
+F 3 "" H 9500 5600 50  0001 C CNN
+	1    9500 5600
+	1    0    0    -1
+$EndComp
+$Comp
+L Mechanical:MountingHole H4
+U 1 1 60D25AB2
+P 10800 6350
+F 0 "H4" H 10700 6304 50  0000 R CNN
+F 1 "MountingHole" H 10700 6395 50  0000 R CNN
+F 2 "MountingHole:MountingHole_2.7mm_M2.5_Pad_Via" H 10800 6350 50  0001 C CNN
+F 3 "~" H 10800 6350 50  0001 C CNN
+	1    10800 6350
+	1    0    0    1
+$EndComp
+$Comp
+L Mechanical:MountingHole H2
+U 1 1 60D4B862
+P 10050 6350
+F 0 "H2" H 9950 6304 50  0000 R CNN
+F 1 "MountingHole" H 9950 6395 50  0000 R CNN
+F 2 "MountingHole:MountingHole_2.7mm_M2.5_Pad_Via" H 10050 6350 50  0001 C CNN
+F 3 "~" H 10050 6350 50  0001 C CNN
+	1    10050 6350
+	1    0    0    1
+$EndComp
+$Comp
+L Mechanical:MountingHole H3
+U 1 1 60D4BDB5
+P 10800 6100
+F 0 "H3" H 10700 6054 50  0000 R CNN
+F 1 "MountingHole" H 10700 6145 50  0000 R CNN
+F 2 "MountingHole:MountingHole_2.7mm_M2.5_Pad_Via" H 10800 6100 50  0001 C CNN
+F 3 "~" H 10800 6100 50  0001 C CNN
+	1    10800 6100
+	1    0    0    1
+$EndComp
+$Comp
+L Mechanical:MountingHole H1
+U 1 1 60D4C572
+P 10050 6100
+F 0 "H1" H 9950 6054 50  0000 R CNN
+F 1 "MountingHole" H 9950 6145 50  0000 R CNN
+F 2 "MountingHole:MountingHole_2.7mm_M2.5_Pad_Via" H 10050 6100 50  0001 C CNN
+F 3 "~" H 10050 6100 50  0001 C CNN
+	1    10050 6100
+	1    0    0    1
+$EndComp
 $EndSCHEMATC

Commit message: 2.2.0
Parts:
- added J21: Conn_02x04_Odd_Even, Connector_PinSocket_2.54mm:PinSocket_2x04_P2.54mm_Vertical, symbol Connector_Generic:Conn_02x04_Odd_Even
- added J22: Conn_01x02_Male, Connector_PinHeader_2.54mm:PinHeader_1x02_P2.54mm_Vertical, symbol Connector:Conn_01x02_Male
Connections:
- net GND: now also J21.2 (Pin_2), J22.2 (Pin_2)
- net RST: now also J21.5 (Pin_5), J21.6 (Pin_6), J22.1 (Pin_1)
- net RXD3v3: now also J21.8 (Pin_8)
- net TXD: now also J21.1 (Pin_1)
- net 3v3: now reaches C1.1, D2.1 (K), U5.2 (VCC)
- net 3v3: now also J21.3 (Pin_3), J21.4 (Pin_4), J21.7 (Pin_7)
Changed lines of the file:
@@
 	1    0    0    1
 $EndComp
+$Comp
+L Connector_Generic:Conn_02x04_Odd_Even J21
+U 1 1 60D18AFC
+P 8250 6000
+F 0 "J21" H 8300 6317 50  0000 C CNN
+F 1 "Conn_02x04_Odd_Even" H 8300 6226 50  0000 C CNN
+F 2 "Connector_PinSocket_2.54mm:PinSocket_2x04_P2.54mm_Vertical" H 8250 6000 50  0001 C CNN
+F 3 "~" H 8250 6000 50  0001 C CNN
+	1    8250 6000
+	1    0    0    -1
+$EndComp
+Text GLabel 8500 1500 3    50   Input ~ 0
+3v3
+Text GLabel 8050 6200 0    50   Input ~ 0
+3v3
+$Comp
+L power:GND #PWR0148
+U 1 1 60D1C882
+P 8900 5900
+F 0 "#PWR0148" H 8900 5650 50  0001 C CNN
+F 1 "GND" H 8900 5750 50  0000 C CNN
+F 2 "" H 8900 5900 50  0001 C CNN
+F 3 "" H 8900 5900 50  0001 C CNN
+	1    8900 5900
+	1    0    0    -1
+$EndComp
+Text GLabel 8050 5900 0    50   Input ~ 0
+TXD
+Text GLabel 8550 6200 2    50   Input ~ 0
+RXD3v3
+Text GLabel 8050 6000 0    50   Input ~ 0
+3v3
+Text GLabel 8550 6000 2    50   Input ~ 0
+3v3
+Wire Wire Line
+	8550 5900 8900 5900
+Text GLabel 8050 6100 0    50   Input ~ 0
+RST
+Text GLabel 8550 6100 2    50   Input ~ 0
+RST
+$Comp
+L Connector:Conn_01x02_Male J22
+U 1 1 60E01238
+P 1300 7250
+F 0 "J22" H 1408 7431 50  0000 C CNN
+F 1 "Conn_01x02_Male" H 1408 7340 50  0000 C CNN
+F 2 "Connector_PinHeader_2.54mm:PinHeader_1x02_P2.54mm_Vertical" H 1300 7250 50  0001 C CNN
+F 3 "~" H 1300 7250 50  0001 C CNN
+	1    1300 7250
+	1    0    0    -1
+$EndComp
+Text GLabel 1500 7250 2    50   Input ~ 0
+RST
+$Comp
+L power:GND #PWR0149
+U 1 1 60E018B0
+P 1500 7350
+F 0 "#PWR0149" H 1500 7100 50  0001 C CNN
+F 1 "GND" H 1505 7177 50  0000 C CNN
+F 2 "" H 1500 7350 50  0001 C CNN
+F 3 "" H 1500 7350 50  0001 C CNN
+	1    1500 7350
+	1    0    0    -1
+$EndComp
 $EndSCHEMATC
