File: g2.kicad_pcb (KiCad board)
At the start: 2 copper layers, 105 x 123 mm, 80 parts, among them J1 USB_B_Micro, J10 Screw, J11 Screw, J12 A, J13 Micro, J14 Speaker, J15 A, J16 A, J17 i2c, J18 i2c, J19 Micro, J2 Screw_Terminal_01x04, J20 Micro, J21 Conn_02x04_Odd_Even, J22 Conn_01x02_Male, J3 Screw, J4 pwm, J5 pwm, J6 pwm, J7 Screw, J8 Screw, J9 Screw, K1 SRD, K2 SRD, K3 SRD, K4 SRD, K5 SRD, K6 SRD, Q1 2N3904, Q2 2N3904, Q3 2N3904, Q4 2N3904, Q5 2N3904, Q6 2N3904, U1 PC817, U2 PC817, U3 PC817, U4 ATmega328P-PU, U5 Sim800l, U6 PC817, U7 PC817, U8 PC817, U9 LD1117S33TR_SOT223, Y1 Crystal

Commit message: with_timer
Parts:
- added J23: i2c, Connector_PinSocket_2.54mm:PinSocket_1x04_P2.54mm_Vertical, F.Cu at (107.7, 53.8)
- added J24: A, Connector_PinHeader_2.54mm:PinHeader_1x03_P2.54mm_Vertical, F.Cu at (116.6, 124.7)
- added J25: A, Connector_PinHeader_2.54mm:PinHeader_1x03_P2.54mm_Vertical, F.Cu at (68.8, 119.1)
- added R17: R_Small, Resistor_THT:R_Axial_DIN0204_L3.6mm_D1.6mm_P5.08mm_Horizontal, F.Cu at (99.8, 41.7)
- added R18: R_Small, Resistor_THT:R_Axial_DIN0204_L3.6mm_D1.6mm_P5.08mm_Horizontal, F.Cu at (103.6, 41.7)
- moved J18 4.57 mm to (107.7, 49.3)
- moved R3 1.14 mm to (81.0, 60.1)
Connections:
- U6 pad 2: D14 -> D014
Routing:
- net Net-(J24-Pad2): track 0.00 -> 53.5 mm
- net +5V: track 494.5 -> 541.4 mm
- net SCL: track 33.1 -> 51.4 mm
- net SDA: track 36.0 -> 49.5 mm
- net D014: track 0.00 -> 5.11 mm
- net D14: track 26.4 -> 21.7 mm
- net P15: track 38.6 -> 34.2 mm
- net MOSI: track 34.9 -> 32.4 mm
- net P16: track 33.8 -> 33.3 mm

Commit message: final
Parts:
- added J26: Conn_01x03_Female, Connector_PinSocket_2.54mm:PinSocket_1x03_P2.54mm_Vertical, F.Cu at (89.2, 77.8)
- moved K4 19.1 mm to (59.3, 133.5)
- moved C6 19.1 mm to (104.6, 100.9)
- moved D5 19.1 mm to (63.8, 133.1)
- moved J15 19.1 mm to (127.7, 87.2)
- moved J16 19.1 mm to (127.7, 91.5)
- moved J2 19.1 mm to (130.6, 98.1)
- moved C2 19.1 mm to (78.6, 34.9)
- moved D8 19.1 mm to (80.1, 44.6)
- moved K2 19.1 mm to (59.3, 98.1)
- moved K6 19.1 mm to (59.3, 46.1)
- moved R1 19.1 mm to (66.9, 85.3)
- moved R15 19.1 mm to (67.9, 39.7)
- moved R6 19.1 mm to (66.9, 102.7)
- moved R7 19.1 mm to (66.9, 120.6)
- moved R8 19.1 mm to (66.9, 137.9)
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- renumbered J17 to Je
Routing:
- net TXD: track 52.7 -> 57.9 mm
- net RST: track 83.5 -> 87.2 mm
