File: g2.sch (KiCad schematic (older format))
At the start: 80 parts, among them J1 USB_B_Micro, J10 Screw, J11 Screw, J12 A, J13 Micro, J14 Speaker, J15 A, J16 A, J17 i2c, J18 i2c, J19 Micro, J2 Screw_Terminal_01x04, J20 Micro, J21 Conn_02x04_Odd_Even, J22 Conn_01x02_Male, J3 Screw, J4 pwm, J5 pwm, J6 pwm, J7 Screw, J8 Screw, J9 Screw, K1 SRD, K2 SRD, K3 SRD, K4 SRD, K5 SRD, K6 SRD, Q1 2N3904, Q2 2N3904, Q3 2N3904, Q4 2N3904, Q5 2N3904, Q6 2N3904, U1 PC817, U2 PC817, U3 PC817, U4 ATmega328P-PU, U5 Sim800l, U6 PC817, U7 PC817, U8 PC817, U9 LD1117S33TR_SOT223, Y1 Crystal

Commit message: with_timer
Parts:
- added J23: i2c, Connector_PinSocket_2.54mm:PinSocket_1x04_P2.54mm_Vertical, symbol Connector:Conn_01x04_Female
- added J24, J25: A, Connector_PinHeader_2.54mm:PinHeader_1x03_P2.54mm_Vertical, symbol Connector:Conn_01x03_Male
- added R17, R18: R_Small, Resistor_THT:R_Axial_DIN0204_L3.6mm_D1.6mm_P5.08mm_Horizontal, symbol Device:R_Small
Connections:
- net +5V: now also J23.3 (Pin_3), J24.1 (Pin_1), R17.1, R18.1
- net D14: now also J25.3 (Pin_3); no longer U6.2
- net GND: now also J23.4 (Pin_4), J24.3 (Pin_3)
- net SCL: now also J23.1 (Pin_1), R18.2
- net SDA: now also J23.2 (Pin_2), R17.2
- new net: J24.2 (Pin_2), J25.1 (Pin_1)
- new net D014: J25.2 (Pin_2), U6.2
Changed lines of the file:
@@
 	2750 5250 2750 5300
 Text GLabel 950  6300 0    50   Input ~ 0
-D14
+D014
 Wire Wire Line
 	1050 6300 950  6300
@@
 Text GLabel 8550 6000 2    50   Input ~ 0
 33v
+$Comp
+L Connector:Conn_01x04_Female J23
+U 1 1 60F568FA
+P 11000 750
+F 0 "J23" H 11028 726 50  0000 L CNN
+F 1 "i2c" H 11028 635 50  0000 L CNN
+F 2 "Connector_PinSocket_2.54mm:PinSocket_1x04_P2.54mm_Vertical" H 11000 750 50  0001 C CNN
+F 3 "~" H 11000 750 50  0001 C CNN
+	1    11000 750
+	1    0    0    -1
+$EndComp
+$Comp
+L power:GND #PWR0152
+U 1 1 60F56900
+P 10650 1000
+F 0 "#PWR0152" H 10650 750 50  0001 C CNN
+F 1 "GND" H 10655 827 50  0000 C CNN
+F 2 "" H 10650 1000 50  0001 C CNN
+F 3 "" H 10650 1000 50  0001 C CNN
+	1    10650 1000
+	1    0    0    -1
+$EndComp
+$Comp
+L power:+5V #PWR0153
+U 1 1 60F56906
+P 10500 850
+F 0 "#PWR0153" H 10500 700 50  0001 C CNN
+F 1 "+5V" H 10515 1023 50  0000 C CNN
+F 2 "" H 10500 850 50  0001 C CNN
+F 3 "" H 10500 850 50  0001 C CNN
+	1    10500 850
+	1    0    0    -1
+$EndComp
+Wire Wire Line
+	10800 950  10650 950
+Wire Wire Line
+	10650 950  10650 1000
+Wire Wire Line
+	10800 850  10500 850
+Text GLabel 10800 750  0    50   Input ~ 0
+SDA
+Text GLabel 10800 650  0    50   Input ~ 0
+SCL
+Text GLabel 9450 2350 0    50   Input ~ 0
+SDA
+Text GLabel 9450 2550 0    50   Input ~ 0
+SCL
+$Comp
+L power:+5V #PWR0154
+U 1 1 60F70456
+P 9950 2300
+F 0 "#PWR0154" H 9950 2150 50  0001 C CNN
+F 1 "+5V" H 9965 2473 50  0000 C CNN
+F 2 "" H 9950 2300 50  0001 C CNN
+F 3 "" H 9950 2300 50  0001 C CNN
+	1    9950 2300
+	1    0    0    -1
+$EndComp
+$Comp
+L Device:R_Small R17
+U 1 1 60F70C5D
+P 9650 2350
+F 0 "R17" V 9454 2350 50  0000 C CNN
+F 1 "R_Small" V 9545 2350 50  0000 C CNN
+F 2 "Resistor_THT:R_Axial_DIN0204_L3.6mm_D1.6mm_P5.08mm_Horizontal" H 9650 2350 50  0001 C CNN
+F 3 "~" H 9650 2350 50  0001 C CNN
+	1    9650 2350
+	0    1    1    0
+$EndComp
+$Comp
+L Device:R_Small R18
+U 1 1 60F72425
+P 9650 2550
+F 0 "R18" V 9454 2550 50  0000 C CNN
+F 1 "R_Small" V 9545 2550 50  0000 C CNN
+F 2 "Resistor_THT:R_Axial_DIN0204_L3.6mm_D1.6mm_P5.08mm_Horizontal" H 9650 2550 50  0001 C CNN
+F 3 "~" H 9650 2550 50  0001 C CNN
+	1    9650 2550
+	0    1    1    0
+$EndComp
+Wire Wire Line
+	9450 2350 9550 2350
+Wire Wire Line
+	9750 2350 9950 2350
+Wire Wire Line
+	9950 2350 9950 2300
+Wire Wire Line
+	9450 2550 9550 2550
+Wire Wire Line
+	9750 2550 9950 2550
+Wire Wire Line
+	9950 2550 9950 2350
+Connection ~ 9950 2350
+$Comp
+L Connector:Conn_01x03_Male J24
+U 1 1 60FCC195
+P 8700 4600
+F 0 "J24" H 8750 4850 50  0000 C CNN
+F 1 "A" H 8750 4800 50  0000 C CNN
+F 2 "Connector_PinHeader_2.54mm:PinHeader_1x03_P2.54mm_Vertical" H 8700 4600 50  0001 C CNN
+F 3 "~" H 8700 4600 50  0001 C CNN
+	1    8700 4600
+	1    0    0    -1
+$EndComp
+$Comp
+L power:+5V #PWR0155
+U 1 1 60FCC19B
+P 8900 4500
+F 0 "#PWR0155" H 8900 4350 50  0001 C CNN
+F 1 "+5V" H 8915 4673 50  0000 C CNN
+F 2 "" H 8900 4500 50  0001 C CNN
+F 3 "" H 8900 4500 50  0001 C CNN
+	1    8900 4500
+	1    0    0    -1
+$EndComp
+$Comp
+L power:GND #PWR0156
+U 1 1 60FCC1A1
+P 8900 4700
+F 0 "#PWR0156" H 8900 4450 50  0001 C CNN
+F 1 "GND" H 8905 4527 50  0000 C CNN
+F 2 "" H 8900 4700 50  0001 C CNN
+F 3 "" H 8900 4700 50  0001 C CNN
+	1    8900 4700
+	1    0    0    -1
+$EndComp
+$Comp
+L Connector:Conn_01x03_Male J25
+U 1 1 60FEDB66
+P 9450 4300
+F 0 "J25" H 9500 4550 50  0000 C CNN
+F 1 "A" H 9500 4500 50  0000 C CNN
+F 2 "Connector_PinHeader_2.54mm:PinHeader_1x03_P2.54mm_Vertical" H 9450 4300 50  0001 C CNN
+F 3 "~" H 9450 4300 50  0001 C CNN
+	1    9450 4300
+	-1   0    0    1
+$EndComp
+Text GLabel 9250 4200 0    50   Input ~ 0
+D14
+Text GLabel 9250 4300 0    50   Input ~ 0
+D014
+Wire Wire Line
+	8900 4600 9250 4600
+Wire Wire Line
+	9250 4600 9250 4400
 $EndSCHEMATC

Commit message: final
Parts:
- added J26: Serial, Connector_PinSocket_2.54mm:PinSocket_1x03_P2.54mm_Vertical, symbol Connector:Conn_01x03_Female
- H1, H2, H3, H4: value MountingHole -> Hole
- J2: value Screw_Terminal_01x04 -> D_I
- J21: value Conn_02x04_Odd_Even -> Esp-01
- J22: value Conn_01x02_Male -> rst btn
- J24: value A -> PIR
- J25: value A -> r
- U9: value LD1117S33TR_SOT223 -> 3v3 regulator
Connections:
- net RST: now also J26.1 (Pin_1)
- net RXD: now also J26.3 (Pin_3)
- net TXD: now also J26.2 (Pin_2)
Other:
- note added: "Alimentation"
- note added: "Circuit De Communication"
- note added: "Circuit Des Relais"
- note added: "Connecteurs Entrée/Sortie"
- note added: "I2C I/O"
- note added: "Microcontrôleur"
- moved on the sheet: C1, C2, C3, C4, C5, C6, C7, C8, D1, D2, D3, D4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
